File: pcb/mppcSensor.kicad_pcb (KiCad board)
At the start: 2 copper layers, 12.7 x 6.3 mm, 4 parts, among them J1 Conn_Coaxial

Commit message: Updated readme with new design, added renderings.
Other:
- board text added: "D1 H1 H2"
Changed lines of the file:
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@@
   (general
     (thickness 1.6)
-    (drawings 8)
+    (drawings 9)
     (tracks 11)
     (zones 0)
@@
     (43 Eco2.User user)
     (44 Edge.Cuts user)
-    (45 Margin user)
+    (45 Margin user hide)
     (46 B.CrtYd user)
     (47 F.CrtYd user)
@@
       (effects (font (size 0.8 0.8) (thickness 0.1)) (justify mirror))
     )
-    (fp_text value Conn_Coaxial (at 0.475 -3.2 270) (layer B.Fab)
+    (fp_text value Conn_Coaxial (at 5 0) (layer B.Fab)
       (effects (font (size 1 1) (thickness 0.15)) (justify mirror))
     )
@@
       (effects (font (size 0.8 0.8) (thickness 0.1)))
     )
-    (fp_text value S13360-2050VE (at 0 2.5) (layer F.Fab)
+    (fp_text value S13360-2050VE (at 0 4.445) (layer F.Fab)
       (effects (font (size 1 1) (thickness 0.15)))
     )
@@
       (effects (font (size 1 1) (thickness 0.15)))
     )
-    (fp_text value MountingHole (at 0 2.9) (layer F.Fab)
-      (effects (font (size 1 1) (thickness 0.15)))
-    )
-    (fp_text user %R (at 0.3 0) (layer F.Fab)
-      (effects (font (size 1 1) (thickness 0.15)))
-    )
+    (fp_text value MountingHole (at 3.23 6.35) (layer F.Fab)
+      (effects (font (size 1 1) (thickness 0.15)))
+    )
+    (fp_circle (center 0 0) (end 2.15 0) (layer F.CrtYd) (width 0.05))
     (fp_circle (center 0 0) (end 1.9 0) (layer Cmts.User) (width 0.15))
-    (fp_circle (center 0 0) (end 2.15 0) (layer F.CrtYd) (width 0.05))
+    (fp_text user %R (at 0.055 0) (layer F.Fab)
+      (effects (font (size 1 1) (thickness 0.15)))
+    )
     (pad 1 thru_hole circle (at 0 0) (size 3.8 3.8) (drill 2.2) (layers *.Cu *.Mask))
   )
@@
       (effects (font (size 1 1) (thickness 0.15)))
     )
-    (fp_text value MountingHole (at 0 2.9) (layer F.Fab)
+    (fp_text value MountingHole (at -5.77 8) (layer F.Fab)
       (effects (font (size 1 1) (thickness 0.15)))
     )
     (fp_circle (center 0 0) (end 2.15 0) (layer F.CrtYd) (width 0.05))
     (fp_circle (center 0 0) (end 1.9 0) (layer Cmts.User) (width 0.15))
-    (fp_text user %R (at 0.3 0) (layer F.Fab)
+    (fp_text user %R (at -0.055 0) (layer F.Fab)
       (effects (font (size 1 1) (thickness 0.15)))
     )
     (pad 1 thru_hole circle (at 0 0) (size 3.8 3.8) (drill 2.2) (layers *.Cu *.Mask))
   )
+  (gr_text "D1\nH1\nH2" (at -8.255 6.35) (layer F.Fab)
+    (effects (font (size 1 1) (thickness 0.2)))
+  )
   (gr_line (start 6.35 3.175) (end 6.35 -3.175) (layer Edge.Cuts) (width 0.15))
