File: pcb/mppcSensor - OSHPark.kicad_pcb (KiCad board)
At the start: 2 copper layers, 13.6 x 4.5 mm, 3 parts, among them J1 Conn_Coaxial

Commit message: oldBoard snapshot
Other:
- board size 13.6 x 4.5 mm -> 13.6 x 6.3 mm
Changed lines of the file:
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@@
   (general
     (thickness 1.6)
-    (drawings 9)
+    (drawings 12)
     (tracks 11)
     (zones 0)
@@
     (pad 1 thru_hole circle (at 0 0) (size 3.8 3.8) (drill 2.2) (layers *.Cu *.Mask))
   )
+  (gr_line (start -6.8 -4.1) (end -6.8 -2.25) (layer Edge.Cuts) (width 0.15))
+  (gr_line (start -5.75 -4.1) (end -6.8 -4.1) (layer Edge.Cuts) (width 0.15))
+  (gr_line (start -5.75 -2.25) (end -5.75 -4.1) (layer Edge.Cuts) (width 0.15))
   (gr_text "D1\nH1\nH2" (at -8.255 6.35) (layer F.Fab)
     (effects (font (size 1 1) (thickness 0.2)))
@@
   (gr_line (start -6.8 2.25) (end 6.8 2.25) (layer Edge.Cuts) (width 0.15))
   (gr_line (start -6.8 -2.25) (end -6.8 2.25) (layer Edge.Cuts) (width 0.15))
-  (gr_line (start 6.8 -2.25) (end -6.8 -2.25) (layer Edge.Cuts) (width 0.15))
+  (gr_line (start 6.8 -2.25) (end -5.75 -2.25) (layer Edge.Cuts) (width 0.15))
   (gr_line (start 1.1 -2.5) (end 1.1 2.5) (layer F.CrtYd) (width 0.15))
   (gr_line (start 6.1 -2.5) (end 1.1 -2.5) (layer F.CrtYd) (width 0.15))
