File: pcb/mppcSensor.sch (KiCad schematic (older format))
At the start: 4 parts, among them J1 Conn_Coaxial

Commit message: oldBoard snapshot
Parts:
- removed H2: MountingHole, MountingHole:MountingHole_2.2mm_M2_ISO14580_Pad, symbol Mechanical:MountingHole
Changed lines of the file:
@@
 EESchema Schematic File Version 4
 LIBS:mppcSensor-cache
-EELAYER 26 0
+EELAYER 29 0
 EELAYER END
 $Descr User 5197 5197
@@
 	1    0    0    -1
 $EndComp
-$Comp
-L Mechanical:MountingHole H2
-U 1 1 5C710D04
-P 800 1000
-F 0 "H2" H 900 1046 50  0000 L CNN
-F 1 "MountingHole" H 900 955 50  0000 L CNN
-F 2 "MountingHole:MountingHole_2.2mm_M2_ISO14580_Pad" H 800 1000 50  0001 C CNN
-F 3 "~" H 800 1000 50  0001 C CNN
-	1    800  1000
-	1    0    0    -1
-$EndComp
